File: blackpill/kint.kicad_sch (KiCad schematic)
At the start: 19 parts, among them J1 THUMB_RIGHT_SPC_KB600, J2 LEFT_13_LT, J3 TOP_LEFT, J4 TOP_RIGHT, J5 THUMB_LEFT_BAK, J6 THUMB_RIGHT_SPC, J7 RIGHT_13_DOWN, J8 THUMB_LEFT_BAK_KB600, U1 YAAJ_WeAct_BlackPill_Part_Lik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

Commit message: Update to remove the need to connect center pins
Connections:
- net 3V3: now also U1.20 (3V3); no longer U1.44 (3V3)
